File: mainBoard/cantact.kicad_pcb (KiCad board)
At the start: 2 copper layers, 36.1 x 59.9 mm, 44 parts, among them J1 Cantact, P2 SWD, P4 USB_C_Plug_USB2.0, U1 STM32F042C6T6, U3 MCP2551-I/SN, U4 XC6220B331MR-G, Y1 16 Mhz

Commit message: feat(Hw):Update_Route_And_Labels
Parts:
- removed the G*** at (150.2, 138.3)
- removed the G*** at (142.5, 122.7)
- removed REF**: OSHW-Logo2_7.3x6mm_SilkScreen, Symbol:OSHW-Logo2_7.3x6mm_SilkScreen
- removed kibuzzard-67FD8E9C: G***, kibuzzard-67FD8E9C
- removed kibuzzard-67FD8EBA: G***, kibuzzard-67FD8EBA
- removed kibuzzard-67FE8A9D (x2): G***, kibuzzard-67FE8A9D
- removed kibuzzard-6802DBB7: G***, kibuzzard-6802DBB7
- added ?: VAL**, Mounting_Holes:MountingHole_2-5mm, F.Cu at (156.2, 113.3)
- added ?: VAL**, Mounting_Holes:MountingHole_2-5mm, F.Cu at (128.5, 147.9)
- added G***: LOGO, Aesthetics:electronic_cats_logo_8x6, F.Cu at (131.4, 140.4)
- added G***: LOGO, Aesthetics:electronic_cats_logo_8x6, B.Cu at (142.4, 116.2)
- added kibuzzard-68FBE69F: G***, kibuzzard-68FBE69F, F.Cu at (154.5, 100.5)
- added kibuzzard-68FBE702: G***, kibuzzard-68FBE702, F.Cu at (142.3, 113.2)
- added kibuzzard-68FBE735: G***, kibuzzard-68FBE735, B.Cu at (142.4, 122.0)
- added kibuzzard-68FBEE71: G***, kibuzzard-68FBEE71, F.Cu at (155.6, 124.3)
- added kibuzzard-68FBEEA6: G***, kibuzzard-68FBEEA6, F.Cu at (155.6, 133.6)
- moved C14 13.2 mm to (148.8, 135.8), turned to 90 degrees
- moved U4 12.3 mm to (146.1, 135.8), turned to 180 degrees
- moved C15 11.8 mm to (143.2, 135.8), turned to 90 degrees
- moved F1 10.4 mm to (146.3, 142.1)
- moved C17 9.53 mm to (146.3, 140.6)
- moved R11 8.92 mm to (144.1, 141.3)
- moved P4 8.92 mm to (142.3, 145.1)
- moved R10 8.19 mm to (140.3, 142.2), turned to 0 degrees
- moved JP1 8.15 mm to (157.9, 124.2)
- moved P2 8.15 mm to (157.9, 133.7)
- moved R1 8.15 mm to (153.9, 124.6)
- moved C11 4.84 mm to (139.6, 136.5)
- moved C12 4.77 mm to (139.9, 134.8)
- moved C2 4.65 mm to (144.2, 123.2)
- moved C4 4.65 mm to (125.9, 131.7)
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Routing:
- net GND: track 58.9 -> 30.2 mm, vias 51 -> 46
- net +5V: track 42.4 -> 26.9 mm
- net /D-: track 12.4 -> 19.6 mm
- net Net-(F1-Pad1): track 20.4 -> 13.3 mm
- net /D+: track 12.7 -> 19.8 mm
- net /LED_GREEN: track 34.7 -> 29.9 mm
- net /CAN+: track 29.4 -> 25.4 mm
- net /CAN-: track 29.3 -> 25.3 mm
- net /SWCLK: track 24.8 -> 21.1 mm
- net /SWDIO: track 26.0 -> 22.9 mm
- net Net-(JP1-Pin_2): track 22.4 -> 25.0 mm
- net /LED_RED: track 43.0 -> 40.8 mm
- net /NRST: track 29.2 -> 27.8 mm
- net +3V3: track 139.5 -> 138.6 mm, vias 5 -> 3
